File: PCB/FreeX.kicad_pcb (KiCad board)
At the start: 2 copper layers, 40 parts, among them J1 2-1734839-4, J2 TF31-6S-0.5SH_800_, J3 USB4105-GF-A, J4 TF31-6S-0.5SH_800_, J5 TF31-6S-0.5SH_800_, Q1 BC817, Q2 BC817, U1 W25Q32JVZPIQ, U2 MPU-9250, U3 ESP32-D0WDQ6, U4 CP2102, U5 TC2014-3.3VxCTTR, U6 LM358PW, U7 TDA7052AT_N2, Y1 ECS-400-10-36-CKY-TR

Commit message: 19th March 2025
Parts:
- removed C3, C4: 12pf, Capacitor_SMD:C_0201_0603Metric
- removed R11, R4, R8: 10K, Resistor_SMD:R_0201_0603Metric
- added C14: 1uF, Capacitor_SMD:C_0201_0603Metric, F.Cu at (119.5, 38.0)
- added C15: 10uF, Capacitor_SMD:C_0201_0603Metric, F.Cu at (86.0, 33.0)
- added C16: 1uF, Capacitor_SMD:C_0201_0603Metric, F.Cu at (102.5, 27.0)
- added C17: 100nF, Capacitor_SMD:C_0201_0603Metric, F.Cu at (112.5, 33.5)
- added C18: 3nF, Capacitor_SMD:C_0201_0603Metric, F.Cu at (86.0, 23.5)
- added C19: 10nF, Capacitor_SMD:C_0201_0603Metric, F.Cu at (84.0, 24.5)
- added C20: 0.1uF, Capacitor_SMD:C_0201_0603Metric, F.Cu at (102.5, 25.5)
- added MK1: CMEJ-0413-42-SMT-TR, CMEJ-0413-42-SMT-TR-ELECTRET-MIC:CMEJ-0413-42-SMT-TR-ELECTRET-MIC, F.Cu at (112.0, 41.5)
- added R12: 1.65K, Resistor_SMD:R_0201_0603Metric, F.Cu at (110.0, 34.5)
- added R13: 100K, Resistor_SMD:R_0201_0603Metric, F.Cu at (80.5, 43.5)
- added R14: 47K, Resistor_SMD:R_0201_0603Metric, F.Cu at (80.5, 42.5)
- added R15: 2.2K, Resistor_SMD:R_0201_0603Metric, F.Cu at (121.5, 38.0)
- added R16: 100K, Resistor_SMD:R_0201_0603Metric, F.Cu at (120.0, 36.5)
- added R17: 100K, Resistor_SMD:R_0201_0603Metric, F.Cu at (121.0, 36.5)
- added R18: 100K, Resistor_SMD:R_0201_0603Metric, F.Cu at (119.0, 36.5)
- added R19: 10K, Resistor_SMD:R_0201_0603Metric, F.Cu at (122.0, 36.5)
- added R20: 20K, Resistor_SMD:R_0201_0603Metric, F.Cu at (84.0, 23.5)
- added U8: AP2127N-3.3, Package_TO_SOT_SMD:SOT-23, F.Cu at (111.9, 37.0)
- added U9: TPS7A0508PDBZ, Package_TO_SOT_SMD:SOT-23, F.Cu at (110.1, 32.5)
- C7: value 100pF -> 0,1uF
- C8: value 0.1uF -> 1uF
- R10: value 10K -> 1k
- U5: value TC2014-3.3VxCTTR -> LTC4054ES5-4.2; footprint Package_TO_SOT_SMD:SOT-23-5 -> Package_TO_SOT_SMD:TSOT-23-5
- U6: value LM358PW -> LMV358M; footprint LM358PW-Amplifier:LM358PW-Amplifier -> LMV358M_OP_AMP_FOR_MIC:LMV358M_OP_AMP_FOR_MIC
- U7: value TDA7052AT_N2 -> LM4810; footprint TDA7052AT_N2-Amplifier:TDA7052AT_N2-Amplifier -> Package_SO:TSSOP-8_3x3mm_P0.65mm
- moved R10 12.2 mm to (93.5, 37.0), turned to 180 degrees
- moved U6 9.77 mm to (118.5, 41.5), turned to 0 degrees
- moved U7 8.67 mm to (116.0, 33.0)
- moved U5 3.43 mm to (116.1, 37.0)
- moved R7 3.11 mm to (82.5, 43.5), turned to 0 degrees
- moved J4 3.01 mm to (117.5, 26.0)
- moved J2 2.77 mm to (108.2, 26.0)
- moved R9 2.33 mm to (82.5, 42.5), turned to 0 degrees
- moved Q2 0.85 mm to (106.0, 32.4)
- moved R6 0.64 mm to (103.0, 31.3)
- moved R5 0.53 mm to (103.2, 33.0)
Connections:
- net /Button_1 renamed /Button_1/GPIO_16
- net /Button_2 renamed /Button_2/GPIO_17
- net Net-(U3-XTAL_N) renamed /OUT/IN/XTAL_N
- net Net-(U3-XTAL_P) renamed /OUT/IN/XTAL_P
- J1 pad 21: /Button_5 -> Net-(U3-VDET_2)
- J1 pad 22: /Button_3 -> /D4/32K_XP/GPIO_32
- J1 pad 3: Net-(U3-GPIO21) -> /SDA/GPIO_21
- J2 pad 1: unconnected-(J2-Pad1) -> /VDD 3.3V POWER
- J2 pad 2: unconnected-(J2-Pad2) -> GND
- J2 pad 3: unconnected-(J2-Pad3) -> /SDA/GPIO_21
- J2 pad 4: unconnected-(J2-Pad4) -> /SCL/GPIO_22
- J2 pad 5: unconnected-(J2-Pad5) -> /XSHUT_1/GPIO14
- J2 pad 6: unconnected-(J2-Pad6) -> /BUZZER_1/GPIO_12
- J3 pad SH1: unconnected-(J3-SHELL_GND-PadSH1)_2 -> Net-(J3-SHELL_GND-PadSH1)
- J3 pad SH2: unconnected-(J3-SHELL_GND-PadSH1)_0 -> Net-(J3-SHELL_GND-PadSH1)
- J3 pad SH3: unconnected-(J3-SHELL_GND-PadSH1) -> Net-(J3-SHELL_GND-PadSH1)
- J3 pad SH4: unconnected-(J3-SHELL_GND-PadSH1)_1 -> Net-(J3-SHELL_GND-PadSH1)
- J4 pad 1: unconnected-(J4-Pad1) -> /VDD 3.3V POWER
- J4 pad 2: unconnected-(J4-Pad2) -> GND
- J4 pad 3: unconnected-(J4-Pad3) -> /SDA/GPIO_21
- J4 pad 4: unconnected-(J4-Pad4) -> /SCL/GPIO_22
- J4 pad 5: unconnected-(J4-Pad5) -> /XSHUT_1/GPIO13
- J4 pad 6: GND -> /BUZZER_1/GPIO_12
- J5 pad 4: /Button_3 -> unconnected-(J5-Pad4)
- J5 pad 5: /Button_4 -> /LED+
- J5 pad 6: /Button_5 -> /LED-
- R10 pad 1: GND -> Net-(U4-REGIN)
- R10 pad 2: /Button_5 -> /LED+
- U1 pad 8: /PROG_RXD -> /VDD SDIO
- U3 pad 11: /Button_5 -> Net-(U3-VDET_2)
- U3 pad 12: /Button_3 -> /D4/32K_XP/GPIO_32
- U3 pad 13: /Button_4 -> /OP-AMP-OUTPUT_2
- U3 pad 15: unconnected-(U3-GPIO26-Pad15) -> /LM4810/AUDIO/GPIO_26
- U3 pad 17: unconnected-(U3-MTMS-Pad17) -> /BATTERY_STATUS
- U3 pad 18: unconnected-(U3-MTDI-Pad18) -> /BUZZER_1/GPIO_12
- U3 pad 20: unconnected-(U3-MTCK-Pad20) -> /XSHUT_1/GPIO13
- U3 pad 26: unconnected-(U3-VDD_SDIO-Pad26) -> /VDD SDIO
- U3 pad 42: Net-(U3-GPIO21) -> /SDA/GPIO_21
- U3 pad 47: unconnected-(U3-CAP2-Pad47) -> Net-(U3-CAP2)
- U3 pad 48: unconnected-(U3-CAP1-Pad48) -> Net-(U3-CAP1)
- U4 pad 6: unconnected-(U4-VDD-Pad6) -> /CHARGE_STATUS
- U5 pad 1: unconnected-(U5-VIN-Pad1) -> /LED-
- U5 pad 2: unconnected-(U5-GND-Pad2) -> GND
- U5 pad 3: unconnected-(U5-ON/~{OFF}-Pad3) -> /`BATTERY +VE
- U5 pad 4: unconnected-(U5-BP-Pad4) -> Net-(U4-REGIN)
- U5 pad 5: unconnected-(U5-VOUT-Pad5) -> Net-(U5-PROG)
- U6 pad 1: unconnected-(U6-1OUT-Pad1) -> /OP-AMP-OUTPUT
- U6 pad 2: unconnected-(U6-1IN--Pad2) -> Net-(U6-INA-)
- U6 pad 3: unconnected-(U6-1IN+-Pad3) -> /NON-INVERTING
- U6 pad 4: unconnected-(U6-GND-Pad4) -> GND
- U6 pad 8: unconnected-(U6-VCC-Pad8) -> /VDD 3.3V POWER
- U7 pad 1: unconnected-(U7-VP-Pad1) -> /SPEAKER+
- U7 pad 2: unconnected-(U7-IN+-Pad2) -> Net-(U7-VIN1)
- U7 pad 3: unconnected-(U7-GND1-Pad3) -> Net-(U7-BYPASS)
- U7 pad 4: unconnected-(U7-VC-Pad4) -> GND
- U7 pad 5: unconnected-(U7-OUT+-Pad5) -> /VDD 3.3V POWER
- U7 pad 6: unconnected-(U7-GND2-Pad6) -> GND
- U7 pad 7: unconnected-(U7-N.C-Pad7) -> /SPEAKER-
- U7 pad 8: unconnected-(U7-OUT--Pad8) -> /VDD 3.3V POWER
Routing:
- net /VDD 3.3V POWER: track 17.7 -> 109.0 mm, vias 6 -> 17
- net /SDA/GPIO_21: track 3.05 -> 92.4 mm, vias 0 -> 12
- net /OP-AMP-OUTPUT: track 0.00 -> 50.8 mm, vias 0 -> 4
- net Net-(U9-VO): track 5.32 -> 54.0 mm, vias 2 -> 5
- net /LED-: track 0.00 -> 45.0 mm, vias 0 -> 4
- net /BUZZER_1/GPIO_12: track 0.00 -> 43.0 mm, vias 0 -> 4
- net /`BATTERY +VE: track 0.00 -> 41.0 mm
- net /Button_5: track 33.0 -> 0.00 mm, vias 4 -> 0
- net /XSHUT_1/GPIO13: track 0.00 -> 32.3 mm, vias 0 -> 4
- net GND: track 144.9 -> 175.3 mm, vias 15 -> 24
- net /Button_4: track 28.1 -> 0.00 mm, vias 6 -> 0
- net /SCL/GPIO_22: track 66.2 -> 93.6 mm, vias 4 -> 12
- net /Button_3: track 25.4 -> 0.00 mm, vias 3 -> 0
- net /VCC3.3V: track 49.1 -> 74.1 mm, vias 10 -> 12
- net /LM4810/AUDIO/GPIO_26: track 0.00 -> 24.5 mm, vias 0 -> 2
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Other:
- board text added: "+"
- board text added: "+ BATTERY"
- board text added: "-"
- board text added: "SPEAKER"
