File: PCB/FreeX.kicad_sch (KiCad schematic)
At the start: 2 parts, among them U1 W25Q32JVZPIQ, U3 ESP32-D0WDQ6

Commit message: 9th, March 2025
Parts:
- added J1: 2-1734839-4, 2-1734839-4 pin-24:2-1734839-4 pin-24, symbol 2-1734839-4 24-pins:2-1734839-4
- added J2: TF31-6S-0.5SH_800_, TF31-6S-0.5SH_800-6-pins:TF31-6S-0.5SH_800-6-pins, symbol TF31-6S-0.5SH_800-6-pins:TF31-6S-0.5SH_800_
- added J3: USB4105-GF-A, USB4105-GF-A TYPE C:USB4105-GF-A TYPE C, symbol USB4105-GF-A TYPE C:USB4105-GF-A
- added J4: 54-00177, 54-00177-Headphone-Jack:54-00177-Headphone-Jack, symbol 54-00177-Headphone-Jack:54-00177
- added U2: MPU-9250, MPU-9250 SENSOR:MPU-9250 SENSOR, symbol MPU-9250 SENSOR:MPU-9250
- added U4: CP2102, CP2102_USB-to-Serial:CP2102_USB-to-Serial, symbol CP2102_USB-to-Serial:CP2102
- added U5: TC2014-3.3VxCTTR, Package_TO_SOT_SMD:SOT-23-5, symbol Regulator_Linear:TC2014-3.3VxCTTR
- added U6: LM358PW, LM358PW-Amplifier:LM358PW-Amplifier, symbol LM358PW-Amplifier:LM358PW
- added U7: TDA7052AT_N2, TDA7052AT_N2-Amplifier:TDA7052AT_N2-Amplifier, symbol TDA7052AT_N2-Amplifier:TDA7052AT_N2
- added Y1: WE-SPXO_IQXO-791, STP_831056298-Crystal-Oscillator:STP_831056298-Crystal-Oscillator, symbol STP_831056298-Crystal-Oscillator:WE-SPXO_IQXO-791
Connections:
- net GND: now also U3.49 (GND)
- net VDD SDIO: now also U3.40 (U0RXD)
- new net: J1.SH1 (SHIELD), J1.SH2 (SHIELD)
- new net: U2.14 (NC), U2.15 (NC), U2.16 (NC), U2.17 (NC), U2.2 (NC), U2.3 (NC), U2.4 (NC), U2.5 (NC), U2.6 (NC)
- new net: J3.A1_B12 (GND), J3.B1_A12 (GND)
- new net: J3.A4_B9 (VBUS), J3.B4_A9 (VBUS)
- new net: J3.SH1 (SHELL_GND), J3.SH2 (SHELL_GND), J3.SH3 (SHELL_GND), J3.SH4 (SHELL_GND)
- new net: U4.10 (NC), U4.13 (NC), U4.14 (NC), U4.15 (NC), U4.16 (NC), U4.17 (NC), U4.18 (NC), U4.19 (NC), U4.20 (NC), U4.21 (NC), U4.22 (NC)
- new net: U4.29 (GND), U4.3 (GND)
Other:
- moved on the sheet: U1, U3

Commit message: 14th, march. 2025
Parts:
- removed J4: 54-00177, 54-00177-Headphone-Jack:54-00177-Headphone-Jack, symbol 54-00177-Headphone-Jack:54-00177
- removed Y1: WE-SPXO_IQXO-791, STP_831056298-Crystal-Oscillator:STP_831056298-Crystal-Oscillator, symbol STP_831056298-Crystal-Oscillator:WE-SPXO_IQXO-791
- added ANT1: Antenna_Dipole, symbol Device:Antenna_Dipole
- added C1, C2: 15pf, Capacitor_SMD:C_0201_0603Metric, symbol Device:C_Small
- added C10, C11, C6, C8, C9: 0.1uF, Capacitor_SMD:C_0201_0603Metric, symbol Device:C_Small
- added C12, C13: 6.8pF, Capacitor_SMD:C_0201_0603Metric, symbol Device:C_Small
- added C3, C4: 12pf, Capacitor_SMD:C_0201_0603Metric, symbol Device:C_Small
- added C5: 10uF, Capacitor_SMD:C_0201_0603Metric, symbol Device:C_Small
- added C7: 100pF, Capacitor_SMD:C_0201_0603Metric, symbol Device:C_Small
- added J4, J5: TF31-6S-0.5SH_800_, TF31-6S-0.5SH_800-6-pins:TF31-6S-0.5SH_800-6-pins, symbol TF31-6S-0.5SH_800-6-pins:TF31-6S-0.5SH_800_
- added L1: 1.6nH, Inductor_SMD:L_0201_0603Metric, symbol Device:L
- added R1, R2, R3: 4.7K, Resistor_SMD:R_0201_0603Metric, symbol Device:R_US
- added Y1: ECS-400-10-36-CKY-TR, 40 MHz_±10ppm_Crystal_10pF_40_Ohms_4-SMD:ECS-400-10-36-CKY-TR, symbol 40 MHz_±10ppm_Crystal_10pF_40_Ohms_4-SMD:ECS-400-10-36-CKY-TR
Connections:
- net VDD SDIO is gone; now on net PROG_RXD: U1.8 (VCC), U3.40 (U0RXD)
- net GND: now also J1.15, J1.2, J1.8, J3.A1_B12 (GND), J3.B1_A12 (GND), U2.11 (FSYNC), U2.18 (GND), ANT1.1, C1.2, C10.2, C11.2, C13.2, C2.2, C3.2, C4.2, C5.2, C6.2, C7.2, C8.2, C9.2, L1.2, R3.2, Y1.2 (GND), Y1.4 (GND)
- net VCC3.3V: now reaches U3.1 (VDDA), U3.43 (VDDA), U3.46 (VDDA)
- net VCC3.3V: now also U3.19 (VDD3P3_RTC), U3.3 (VDD3P3), U3.37 (VDD3P3_CPU), U3.4 (VDD3P3), C10.1, C5.1, C6.1, C7.1, C8.1, C9.1
- net at U3.10 (VDET_1): now also J1.20
- net at U3.11 (VDET_2): now also J1.21
- net D4/32K_XP/GPIO_32: now reaches U3.12 (32K_XP)
- net D4/32K_XP/GPIO_32: now also J1.22, C3.1
- net at U3.13 (32K_XN): now also C4.1
- net VS/GPIO_25: now reaches U3.14 (GPIO25)
- net VS/GPIO_25: now also J1.7
- net PCLK/GPIO_27: now reaches U3.16 (GPIO27)
- net PCLK/GPIO_27: now also J1.17
- net ANTENNA: now reaches U3.2 (LNA_IN)
- net ANTENNA: now also C12.2, L1.1
- net RESET/MTDO/GPIO 15: now reaches U3.21 (MTDO)
- net RESET/MTDO/GPIO 15: now also J1.6
- net VDD 3.3V POWER: now reaches U3.22 (GPIO2)
- net at U3.23 (GPIO0): now also J1.13
- net INT/GPIO_4: now reaches U3.24 (GPIO4)
- net INT/GPIO_4: now also U2.12 (INT)
- net at U3.34 (GPIO5): now also J1.12
- net D8/GPIO_18: now reaches U3.35 (GPIO18)
- net D8/GPIO_18: now also J1.14
- net HS/GPIO_23: now reaches U3.36 (GPIO23)
- net HS/GPIO_23: now also J1.9
- net D7/GPIO_19: now reaches U3.38 (GPIO19)
- net D7/GPIO_19: now also J1.16
- net SCL/GPIO_22: now reaches U3.39 (GPIO22)
- net SCL/GPIO_22: now also J1.5, U2.23 (SCL/SCLK), R2.1
- net PROG_TXD: now reaches U3.41 (U0TXD)
- net PROG_TXD: now also U4.26 (TXD)
- net at U3.42 (GPIO21): now also J1.3
- net at U3.44 (XTAL_N): now also C2.1, Y1.1 (IN/OUT)
- net at U3.45 (XTAL_P): now also C1.1, Y1.3 (OUT/IN)
- net at U3.5 (SENSOR_VP): now also J1.18
- net at U3.8 (SENSOR_VN): now also J1.19
- net at U2.10 (REGOUT): now also C11.1
- net VDD33: now reaches U2.13 (VDD)
- net VDD33: now also R1.2, R2.2
- net SDA/GPIO_21: now reaches U2.24 (SDA/SDI)
- net SDA/GPIO_21: now also R1.1
- net at U2.9 (AD0/SDO): now also R3.1
- net at J3.A4_B9 (VBUS), J3.B4_A9 (VBUS): now also U4.7 (REGIN), U4.8 (VBUS)
- net at J3.B6 (DP2): now also U4.4 (D+)
- net at J3.B7 (DN2): now also U4.5 (D-)
- net PROG_RXD: now reaches U4.25 (RXD)
- new net: ANT1.2, C12.1, C13.1
- no-connect marks 0 -> 12
Other:
- moved on the sheet: J1, J2, J3, U1, U2, U3, U4, U5, U6

Commit message: 15th, march. 2025
Parts:
- added Q1, Q2: BC817, Package_TO_SOT_SMD:SOT-23, symbol Transistor_BJT:BC817
- added R10, R11, R4, R5, R6, R7, R8, R9: 10K, Resistor_SMD:R_0201_0603Metric, symbol Device:R_US
- added U8: AP2127N-3.3, Package_TO_SOT_SMD:SOT-23, symbol Regulator_Linear:AP2127N-3.3
Connections:
- net D4/32K_XP/GPIO_32 is gone; now on net Button_3: C3.1, J1.22, U3.12 (32K_XP)
- net GND: now also J4.6, U4.29 (GND), U4.3 (GND), R10.1, R11.1, R7.1, R8.1, R9.1
- net VCC3.3V: now also J5.1
- net VDD 3.3V POWER: now also J1.11, J1.4, U2.13 (VDD), R4.2
- net VDD33: no longer U2.13 (VDD)
- net Button_4: now reaches C4.1, U3.13 (32K_XN)
- net Button_4: now also J5.5, R11.2
- net Button_5: now reaches J1.21, U3.11 (VDET_2)
- net Button_5: now also J5.6, R10.2
- net GPIO00: now reaches J1.13, U3.23 (GPIO0)
- net GPIO00: now also Q1.3 (C)
- net Button_1: now reaches U3.25 (GPIO16)
- net Button_1: now also J5.2, R9.2
- net Button_2: now reaches U3.27 (GPIO17)
- net Button_2: now also J5.3, R7.2
- net EN/CHIP_PU: now reaches U3.9 (CHIP_PU)
- net EN/CHIP_PU: now also Q2.3 (C)
- net at J1.10: now also R4.1
- net Button_3: now reaches J5.4
- net Button_3: now also R8.2
- net at U4.24 (RTS): now also Q2.2 (E), R5.2
- net at U4.28 (DTR): now also Q1.2 (E), R6.2
- new net: Q2.1 (B), R6.1
- new net: Q1.1 (B), R5.1
- no-connect marks 12 -> 27
Other:
- moved on the sheet: J2, J3, U4, U5

Commit message: 19th March 2025
Parts:
- removed C3, C4: 12pf, Capacitor_SMD:C_0201_0603Metric, symbol Device:C_Small
- removed R11, R4, R8: 10K, Resistor_SMD:R_0201_0603Metric, symbol Device:R_US
- removed U5: TC2014-3.3VxCTTR, Package_TO_SOT_SMD:SOT-23-5, symbol Regulator_Linear:TC2014-3.3VxCTTR
- removed U6: LM358PW, LM358PW-Amplifier:LM358PW-Amplifier, symbol LM358PW-Amplifier:LM358PW
- removed U7: TDA7052AT_N2, TDA7052AT_N2-Amplifier:TDA7052AT_N2-Amplifier, symbol TDA7052AT_N2-Amplifier:TDA7052AT_N2
- added C14, C16: 1uF, Capacitor_SMD:C_0201_0603Metric, symbol Device:C_Small
- added C15: 10uF, Capacitor_SMD:C_0201_0603Metric, symbol Device:C_Small
- added C17: 100nF, Capacitor_SMD:C_0201_0603Metric, symbol Device:C_Small
- added C18: 3nF, Capacitor_SMD:C_0201_0603Metric, symbol Device:C_Small
- added C19: 10nF, Capacitor_SMD:C_0201_0603Metric, symbol Device:C_Small
- added C20: 0.1uF, Capacitor_SMD:C_0201_0603Metric, symbol Device:C_Small
- added MK1: CMEJ-0413-42-SMT-TR, CMEJ-0413-42-SMT-TR-ELECTRET-MIC:CMEJ-0413-42-SMT-TR-ELECTRET-MIC, symbol CMEJ-0413-42-SMT-TR-ELECTRET-MIC:CMEJ-0413-42-SMT-TR
- added R12: 1.65K, Resistor_SMD:R_0201_0603Metric, symbol Device:R_US
- added R13, R16, R17, R18: 100K, Resistor_SMD:R_0201_0603Metric, symbol Device:R_US
- added R14: 47K, Resistor_SMD:R_0201_0603Metric, symbol Device:R_US
- added R15: 2.2K, Resistor_SMD:R_0201_0603Metric, symbol Device:R_US
- added R19: 10K, Resistor_SMD:R_0201_0603Metric, symbol Device:R_US
- added R20: 20K, Resistor_SMD:R_0201_0603Metric, symbol Device:R_US
- added U5: LTC4054ES5-4.2, Package_TO_SOT_SMD:TSOT-23-5, symbol Battery_Management:LTC4054ES5-4.2
- added U6: LMV358M, LMV358M_OP_AMP_FOR_MIC:LMV358M_OP_AMP_FOR_MIC, symbol LMV358M_OP_AMP_FOR_MIC:LMV358M
- added U7: LM4810, Package_SO:TSSOP-8_3x3mm_P0.65mm, symbol Amplifier_Audio:LM4810
- added U9: TPS7A0508PDBZ, Package_TO_SOT_SMD:SOT-23, symbol Regulator_Linear:TPS7A0508PDBZ
- ANT1: now fitted
- C7: value 100pF -> 0,1uF
- C8: value 0.1uF -> 1uF
- R10: value 10K -> 1k
Connections:
- net GND: now also J2.2, J4.2, U8.1 (GND), C17.1, C19.1, C20.2, MK1.2, R12.1, R14.1, R17.2, R19.2, U5.2 (GND), U6.4 (V-), U7.4 (GND), U7.6 (VIN2), U9.1 (GND); no longer J4.6, R10.1
- net PROG_RXD: no longer U1.8 (VCC)
- net SCL/GPIO_22: now also J2.4, J4.4
- net SDA/GPIO_21: now also J1.3, J2.3, J4.3, U3.42 (GPIO21)
- net VCC3.3V: now also U8.2 (VO)
- net VDD 3.3V POWER: now also J2.1, J4.1, R15.1, R16.1, U6.8 (V+), U7.5 (SHDN), U7.8 (VDD), U9.3 (VI)
- net OUT/IN/XTAL_N: now reaches C2.1, U3.44 (XTAL_N), Y1.1 (IN/OUT)
- net OUT/IN/XTAL_P: now reaches C1.1, U3.45 (XTAL_P), Y1.3 (OUT/IN)
- net XSHUT_1/GPIO14: now reaches J2.5
- net BUZZER_1/GPIO_12: now reaches J2.6
- net BUZZER_1/GPIO_12: now also J4.6, U3.18 (MTDI)
- net at J1.10: now also U9.2 (VO)
- net LM4810/AUDIO/GPIO_26: now reaches U3.15 (GPIO26)
- net LM4810/AUDIO/GPIO_26: now also C16.2
- net BATTERY_STATUS: now reaches U3.17 (MTMS)
- net BATTERY_STATUS: now also R13.1, R14.2
- net XSHUT_1/GPIO13: now reaches U3.20 (MTCK)
- net XSHUT_1/GPIO13: now also J4.5
- net VDD SDIO: now reaches U3.26 (VDD_SDIO)
- net VDD SDIO: now also U1.8 (VCC), C20.1
- net at U3.47 (CAP2): now also C18.1, R20.1
- net at U3.48 (CAP1): now also C18.2, C19.2, R20.2
- net at J3.A4_B9 (VBUS), J3.B4_A9 (VBUS), U4.7 (REGIN)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: now also R10.1, U5.4 (V_{CC})
- net CHARGE_STATUS: now reaches U4.6 (VDD)
- net `BATTERY +VE: now reaches U8.3 (VI)
- net `BATTERY +VE: now also R13.2, U5.3 (BAT)
- net Button_1 renamed Button_1/GPIO_16
- net Button_2 renamed Button_2/GPIO_17
- net Button_3 renamed D4/32K_XP/GPIO_32
- net D4/32K_XP/GPIO_32: no longer J5.4
- net Button_4 renamed LED+
- net LED+: now also R10.2; no longer U3.13 (32K_XN)
- net Button_5: no longer names the net of J1.21, U3.11 (VDET_2)
- net Button_5: no longer J5.6, R10.2
- new net: R18.1, R19.1, U6.2 (INA-)
- new net: C14.1, MK1.1, R15.2
- new net: C17.2, U7.3 (BYPASS)
- new net: R12.2, U5.5 (PROG)
- new net: C16.1, U7.2 (VIN1)
- new net LED-: J5.6, U5.1 (~{CHRG})
- new net NON-INVERTING: C14.2, R16.2, R17.1, U6.3 (INA+)
- new net OP-AMP-OUTPUT: C15.2, R18.2, U6.1 (OUT_A)
- new net OP-AMP-OUTPUT_2: C15.1, U3.13 (32K_XN)
- new net SPEAKER+: U7.1 (VOUT1)
- new net SPEAKER-: U7.7 (VOUT2)
- no-connect marks 27 -> 29
Other:
- moved on the sheet: C1, C10, C11, C12, C13, C2, C5, C6, C7, C8, C9, J2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
